File: pcb/SimpleInterface.kicad_pcb (KiCad board)
At the start: 2 copper layers, 65.5 x 58.4 mm, 19 parts, among them J1 IO Select, J2 IRQ Enable, J3 Microcontroller Port, P1 X16_Card_Edge, Q1 BS170, U1 74ACT04, U2 74ACT00, U3 74ACT02, U4 74AHC273, U5 74LS157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

Commit message: Ambiguous data bus renaming: Bus signals named "CDn" for Client, "HDn" for Host, and "BDn" for Bus.
Parts:
- U5: value 74LS157 -> 74ACT157
- U6: value 74LS245 -> 74ACT245
Connections:
- net /D0 renamed /BD0
- net /D1 renamed /BD1
- net /D2 renamed /BD2
- net /D3 renamed /BD3
- net /D4 renamed /BD4
- net /D5 renamed /BD5
- net /D6 renamed /BD6
- net /D7 renamed /BD7
- net /IN_D0 renamed /C_D0
- net /IN_D1 renamed /C_D1
- net /IN_D2 renamed /C_D2
- net /IN_D3 renamed /C_D3
- net /IN_D4 renamed /C_D4
- net /IN_D5 renamed /C_D5
- net /IN_D6 renamed /C_D6
- net /IN_D7 renamed /C_D7
- net /OUT_D0 renamed /H_D0
- net /OUT_D1 renamed /H_D1
- net /OUT_D2 renamed /H_D2
- net /OUT_D3 renamed /H_D3
- net /OUT_D4 renamed /H_D4
- net /OUT_D5 renamed /H_D5
- net /OUT_D6 renamed /H_D6
- net /OUT_D7 renamed /H_D7
